Commit message: so_arm_100_description: 3. provide valid hardware block
- Provide valid hardware block in so_arm_100_5dof_position.ros2_control.xacro
- Add params to support the SOARM100Interface.
- Set SOARM100System as the ros2_control system name.
- Use correct `use_sim` param in the joint state pub gui launch.

Signed-off-by: Rhys Mainwaring <rhys.mainwaring@me.com>

File: so_arm_100_description/ros2_control/so_arm_100_5dof_position.ros2_control.xacro (robot description, xacro)
@@ -1,33 +1,53 @@
 <?xml version="1.0"?>
 <robot xmlns:xacro="http://www.ros.org/wiki/xacro">
-  <xacro:macro name="so_arm_100_5dof_system" params="name prefix use_sim:=^|false use_topic_hardware_interface:=^|false use_fake_hardware:=^|false">
+  <xacro:macro name="so_arm_100_5dof_system"
+    params="
+      name
+      prefix
+      use_sim:=^|false
+      use_topic_hardware_interface:=^|false
+      use_fake_hardware:=^|false
+      serial_port:=^|/dev/ttyUSB0
+      serial_baudrate:=^|1000000
+      servo_speed:=^|2400
+      servo_acceleration:=^|50">
     <!--
     Parameters
-       name: name given to the controller system
-       prefix: prefix for joints and links
-       use_sim: true if using Gazebo
-       use_topic_hardware_interface: true if using topic based control
-       use_fake_hardware: true if not use_sim and using fake hardware
+        name: name given to the controller system
+        prefix: prefix for joints and links
+        use_sim: true if using Gazebo
+        use_topic_hardware_interface: true if using topic based control
+        use_fake_hardware: true if not use_sim and using fake hardware
+        serial_port: servo controller board serial port
+        serial_baudrate: servo controller board serial baudrate
+        servo_speed: servo move speed in ticks/s
+        servo_acceleration: servo move acceleration in ticks/s^2
     -->
     <ros2_control name="${name}" type="system">
-      <xacro:if value="$(arg use_sim)">
-          <hardware>
-              <xacro:if value="${use_topic_hardware_interface}">
-                  <plugin>joint_state_topic_hardware_interface/JointStateTopicSystem</plugin>
-                  <param name="joint_commands_topic">/robot_joint_commands</param>
-                  <param name="joint_states_topic">/robot_joint_states</param>
-              </xacro:if>
-              <xacro:unless value="$(arg use_topic_hardware_interface)">
-                <plugin>gz_ros2_control/GazeboSimSystem</plugin>
-              </xacro:unless>
-          </hardware>
-      </xacro:if>
-      <xacro:unless value="$(arg use_sim)">
-          <hardware>
-              <xacro:if value="${use_fake_hardware}">
-                <plugin>mock_components/GenericSystem</plugin>
-              </xacro:if>
-          </hardware>
-      </xacro:unless>
+      <hardware>
+        <xacro:if value="$(arg use_sim)">
+          <xacro:if value="${use_topic_hardware_interface}">
+            <plugin>joint_state_topic_hardware_interface/JointStateTopicSystem</plugin>
+            <param name="joint_commands_topic">/robot_joint_commands</param>
+            <param name="joint_states_topic">/robot_joint_states</param>
+          </xacro:if>
+          <xacro:unless value="$(arg use_topic_hardware_interface)">
+            <plugin>gz_ros2_control/GazeboSimSystem</plugin>
+          </xacro:unless>
+        </xacro:if>
+        <xacro:unless value="$(arg use_sim)">
+          <xacro:if value="${use_fake_hardware}">
+            <plugin>mock_components/GenericSystem</plugin>
+          </xacro:if>
+          <xacro:unless value="$(arg use_fake_hardware)">
+            <plugin>so_arm_100_controller/SOARM100Interface</plugin>
+            <param name="use_serial">true</param>
+            <param name="serial_port">${serial_port}</param>
+            <param name="serial_baudrate">${serial_baudrate}</param>
+            <param name="servo_speed">${servo_speed}</param>
+            <param name="servo_acceleration">${servo_acceleration}</param>
+          </xacro:unless>
+        </xacro:unless>
+      </hardware>
       <joint name="${prefix}Shoulder_Rotation">
         <command_interface name="position">

File: so_arm_100_description/urdf/so_arm_100_5dof.urdf.xacro (robot description, xacro)
@@ -28,5 +28,5 @@
   <xacro:include filename="$(find so_arm_100_description)/ros2_control/$(arg ros2_control_type).ros2_control.xacro" />
   <xacro:so_arm_100_5dof_system
-    name="SOARM101System"
+    name="SOARM100System"
     prefix="$(arg prefix)"
     use_sim="$(arg use_sim)"

Commit message: so_arm_100_description: use initial positions file with JointStateTopicsSystem
- Use initial positions file, if present, to initialise the topic based control system.

Signed-off-by: Rhys Mainwaring <rhys.mainwaring@me.com>

File: so_arm_100_description/ros2_control/so_arm_100_5dof_position.ros2_control.xacro (robot description, xacro)
@@ -5,4 +5,5 @@
       name
       prefix
+      initial_positions_file:=^|''
       use_sim:=^|false
       use_topic_hardware_interface:=^|false
@@ -16,4 +17,5 @@
         name: name given to the controller system
         prefix: prefix for joints and links
+        initial_positions_file: initial positions file for joints
         use_sim: true if using Gazebo
         use_topic_hardware_interface: true if using topic based control
@@ -24,4 +26,7 @@
         servo_acceleration: servo move acceleration in ticks/s^2
     -->
+  <xacro:if value="${initial_positions_file != ''}">
+      <xacro:property name="initial_positions" value="${xacro.load_yaml(initial_positions_file)['initial_positions']}"/>
+  </xacro:if>
     <ros2_control name="${name}" type="system">
       <hardware>
@@ -54,4 +59,8 @@
           <param name="min">-3.14</param>
           <param name="max">3.14</param>
+          <xacro:if value="${initial_positions_file != ''}">
+            <xacro:property name="joint_name" value="${prefix}Shoulder_Rotation"/>
+            <param name="initial_value">${initial_positions[joint_name]}</param>
+          </xacro:if>
         </command_interface>
         <state_interface name="position"/>
@@ -63,4 +72,8 @@
           <param name="min">-3.14</param>
           <param name="max">3.14</param>
+          <xacro:if value="${initial_positions_file != ''}">
+            <xacro:property name="joint_name" value="${prefix}Shoulder_Pitch"/>
+            <param name="initial_value">${initial_positions[joint_name]}</param>
+          </xacro:if>
         </command_interface>
         <state_interface name="position"/>
@@ -72,4 +85,8 @@
           <param name="min">-3.14</param>
           <param name="max">3.14</param>
+          <xacro:if value="${initial_positions_file != ''}">
+            <xacro:property name="joint_name" value="${prefix}Elbow"/>
+            <param name="initial_value">${initial_positions[joint_name]}</param>
+          </xacro:if>
         </command_interface>
         <state_interface name="position"/>
@@ -81,4 +98,8 @@
           <param name="min">-3.14</param>
           <param name="max">3.14</param>
+          <xacro:if value="${initial_positions_file != ''}">
+            <xacro:property name="joint_name" value="${prefix}Wrist_Pitch"/>
+            <param name="initial_value">${initial_positions[joint_name]}</param>
+          </xacro:if>
         </command_interface>
         <state_interface name="position"/>
@@ -90,4 +111,8 @@
           <param name="min">-3.14</param>
           <param name="max">3.14</param>
+          <xacro:if value="${initial_positions_file != ''}">
+            <xacro:property name="joint_name" value="${prefix}Wrist_Roll"/>
+            <param name="initial_value">${initial_positions[joint_name]}</param>
+          </xacro:if>
         </command_interface>
         <state_interface name="position"/>
@@ -99,4 +124,8 @@
           <param name="min">-0.1792</param>
           <param name="max">1.57</param>
+          <xacro:if value="${initial_positions_file != ''}">
+            <xacro:property name="joint_name" value="${prefix}Gripper"/>
+            <param name="initial_value">${initial_positions[joint_name]}</param>
+          </xacro:if>
         </command_interface>
         <state_interface name="position"/>
