Commit message: Reorganize repo with SO-100 arm and hardware packages

File: SO-100-arm/so_arm_100_description/gazebo/so_arm_100_5dof.gazebo.xacro (robot description, xacro)
@@ -1,20 +1,11 @@
 <?xml version="1.0"?>
 <robot xmlns:xacro="http://ros.org/wiki/xacro">
-  <xacro:macro name="so_arm_100_5dof_gazebo"
-    params="
-      prefix
-      initial_positions_file:=^|''
-      ros2_controllers_file:=^|''
-      use_topic_hardware_interface:=^|false">
+  <xacro:macro name="so_arm_100_5dof_gazebo" params="prefix ros2_controllers_file:=^|'' use_topic_hardware_interface:=^|false">
   <!--
   Parameters
       prefix: prefix for joints and links
-      initial_positions_file: initial positions file for joints
       ros2_controllers_file: ros2_controller configuration file for gz_ros2_control
       use_topic_hardware_interface: true if using topic based control
   -->
-  <xacro:if value="${initial_positions_file != ''}">
-      <xacro:property name="initial_positions" value="${xacro.load_yaml(initial_positions_file)['initial_positions']}"/>
-  </xacro:if>
   <gazebo>
     <plugin name="gz::sim::systems::JointStatePublisher"
@@ -61,8 +52,4 @@
         <cmd_max>100.0</cmd_max>
         <cmd_min>-100.0</cmd_min>
-        <xacro:if value="${initial_positions_file != ''}">
-          <xacro:property name="joint_name" value="${prefix}Shoulder_Rotation"/>
-          <initial_position>${initial_positions[joint_name]}</initial_position>
-        </xacro:if>
       </plugin>
       <plugin name="gz::sim::systems::JointPositionController"
@@ -77,8 +64,4 @@
         <cmd_max>100.0</cmd_max>
         <cmd_min>-100.0</cmd_min>
-        <xacro:if value="${initial_positions_file != ''}">
-          <xacro:property name="joint_name" value="${prefix}Shoulder_Pitch"/>
-          <initial_position>${initial_positions[joint_name]}</initial_position>
-        </xacro:if>
       </plugin>
       <plugin name="gz::sim::systems::JointPositionController"
@@ -93,8 +76,4 @@
         <cmd_max>100.0</cmd_max>
         <cmd_min>-100.0</cmd_min>
-        <xacro:if value="${initial_positions_file != ''}">
-          <xacro:property name="joint_name" value="${prefix}Elbow"/>
-          <initial_position>${initial_positions[joint_name]}</initial_position>
-        </xacro:if>
       </plugin>
       <plugin name="gz::sim::systems::JointPositionController"
@@ -109,8 +88,4 @@
         <cmd_max>100.0</cmd_max>
         <cmd_min>-100.0</cmd_min>
-        <xacro:if value="${initial_positions_file != ''}">
-          <xacro:property name="joint_name" value="${prefix}Wrist_Pitch"/>
-          <initial_position>${initial_positions[joint_name]}</initial_position>
-        </xacro:if>
       </plugin>
       <plugin name="gz::sim::systems::JointPositionController"
@@ -125,8 +100,4 @@
         <cmd_max>100.0</cmd_max>
         <cmd_min>-100.0</cmd_min>
-        <xacro:if value="${initial_positions_file != ''}">
-          <xacro:property name="joint_name" value="${prefix}Wrist_Roll"/>
-          <initial_position>${initial_positions[joint_name]}</initial_position>
-        </xacro:if>
       </plugin>
       <plugin name="gz::sim::systems::JointPositionController"
@@ -141,8 +112,4 @@
         <cmd_max>100.0</cmd_max>
         <cmd_min>-100.0</cmd_min>
-        <xacro:if value="${initial_positions_file != ''}">
-          <xacro:property name="joint_name" value="${prefix}Gripper"/>
-          <initial_position>${initial_positions[joint_name]}</initial_position>
-        </xacro:if>
       </plugin>
     </xacro:if>

File: SO-100-arm/so_arm_100_description/ros2_control/so_arm_100_5dof_position.ros2_control.xacro (robot description, xacro)
@@ -5,9 +5,8 @@
       name
       prefix
-      initial_positions_file:=^|''
       use_sim:=^|false
       use_topic_hardware_interface:=^|false
       use_fake_hardware:=^|false
-      serial_port:=^|/dev/ttyUSB0
+      serial_port:=^|/dev/ttyACM0
       serial_baudrate:=^|1000000
       servo_speed:=^|2400
@@ -17,5 +16,4 @@
         name: name given to the controller system
         prefix: prefix for joints and links
-        initial_positions_file: initial positions file for joints
         use_sim: true if using Gazebo
         use_topic_hardware_interface: true if using topic based control
@@ -26,7 +24,4 @@
         servo_acceleration: servo move acceleration in ticks/s^2
     -->
-  <xacro:if value="${initial_positions_file != ''}">
-      <xacro:property name="initial_positions" value="${xacro.load_yaml(initial_positions_file)['initial_positions']}"/>
-  </xacro:if>
     <ros2_control name="${name}" type="system">
       <hardware>
@@ -34,6 +29,6 @@
           <xacro:if value="${use_topic_hardware_interface}">
             <plugin>joint_state_topic_hardware_interface/JointStateTopicSystem</plugin>
-            <param name="joint_commands_topic">robot_joint_commands</param>
-            <param name="joint_states_topic">robot_joint_states</param>
+            <param name="joint_commands_topic">/robot_joint_commands</param>
+            <param name="joint_states_topic">/robot_joint_states</param>
           </xacro:if>
           <xacro:unless value="${use_topic_hardware_interface}">
@@ -59,8 +54,4 @@
           <param name="min">-3.14</param>
           <param name="max">3.14</param>
-          <xacro:if value="${initial_positions_file != ''}">
-            <xacro:property name="joint_name" value="${prefix}Shoulder_Rotation"/>
-            <param name="initial_value">${initial_positions[joint_name]}</param>
-          </xacro:if>
         </command_interface>
         <state_interface name="position"/>
@@ -72,8 +63,4 @@
           <param name="min">-3.14</param>
           <param name="max">3.14</param>
-          <xacro:if value="${initial_positions_file != ''}">
-            <xacro:property name="joint_name" value="${prefix}Shoulder_Pitch"/>
-            <param name="initial_value">${initial_positions[joint_name]}</param>
-          </xacro:if>
         </command_interface>
         <state_interface name="position"/>
@@ -85,8 +72,4 @@
           <param name="min">-3.14</param>
           <param name="max">3.14</param>
-          <xacro:if value="${initial_positions_file != ''}">
-            <xacro:property name="joint_name" value="${prefix}Elbow"/>
-            <param name="initial_value">${initial_positions[joint_name]}</param>
-          </xacro:if>
         </command_interface>
         <state_interface name="position"/>
@@ -98,8 +81,4 @@
           <param name="min">-3.14</param>
           <param name="max">3.14</param>
-          <xacro:if value="${initial_positions_file != ''}">
-            <xacro:property name="joint_name" value="${prefix}Wrist_Pitch"/>
-            <param name="initial_value">${initial_positions[joint_name]}</param>
-          </xacro:if>
         </command_interface>
         <state_interface name="position"/>
@@ -111,8 +90,4 @@
           <param name="min">-3.14</param>
           <param name="max">3.14</param>
-          <xacro:if value="${initial_positions_file != ''}">
-            <xacro:property name="joint_name" value="${prefix}Wrist_Roll"/>
-            <param name="initial_value">${initial_positions[joint_name]}</param>
-          </xacro:if>
         </command_interface>
         <state_interface name="position"/>
@@ -124,8 +99,4 @@
           <param name="min">-0.1792</param>
           <param name="max">1.57</param>
-          <xacro:if value="${initial_positions_file != ''}">
-            <xacro:property name="joint_name" value="${prefix}Gripper"/>
-            <param name="initial_value">${initial_positions[joint_name]}</param>
-          </xacro:if>
         </command_interface>
         <state_interface name="position"/>

File: SO-100-arm/so_arm_100_description/urdf/so_arm_100_5dof.urdf.xacro (robot description, xacro)
@@ -2,5 +2,4 @@
 <robot name="so_arm_100_5dof" xmlns:xacro="http://ros.org/wiki/xacro">
   <xacro:arg name="prefix" default="" />
-  <xacro:arg name="initial_positions_file" default="" />
   <xacro:arg name="use_sim" default="false" />
   <xacro:arg name="use_topic_hardware_interface" default="false" />
@@ -23,5 +22,4 @@
       <xacro:so_arm_100_5dof_gazebo
         prefix="$(arg prefix)"
-        initial_positions_file="$(arg initial_positions_file)"
         ros2_controllers_file="$(arg ros2_controllers_file)"
         use_topic_hardware_interface="$(arg use_topic_hardware_interface)" />

File: SO-100-arm/so_arm_100_moveit_config/config/so_arm_100.ros2_control.xacro (robot description, xacro)
@@ -1,5 +1,5 @@
 <?xml version="1.0"?>
 <robot xmlns:xacro="http://www.ros.org/wiki/xacro">
-    <xacro:macro name="so_arm_100_ros2_control" params="name initial_positions_file use_fake_hardware serial_port:=^|/dev/ttyUSB0 serial_baudrate:=^|1000000 servo_speed:=^|2400 servo_acceleration:=^|50" >
+    <xacro:macro name="so_arm_100_ros2_control" params="name initial_positions_file use_fake_hardware serial_port:=^|/dev/ttyACM0 serial_baudrate:=^|1000000 servo_speed:=^|2400 servo_acceleration:=^|50" >
         <xacro:property name="initial_positions" value="${xacro.load_yaml(initial_positions_file)['initial_positions']}"/>
         <ros2_control name="${name}" type="system">

File: SO-100-arm/so_arm_100_moveit_config/config/so_arm_100.urdf.xacro (robot description, xacro)
@@ -4,5 +4,5 @@
     <xacro:arg name="initial_positions_file" default="initial_positions.yaml" />
     <xacro:arg name="use_fake_hardware" default="false"/>
-    <xacro:arg name="serial_port" default="/dev/ttyUSB0"/>
+    <xacro:arg name="serial_port" default="/dev/ttyACM0"/>
     <xacro:arg name="serial_baudrate" default="1000000"/>
     <xacro:arg name="servo_speed" default="2400"/>
